File: Electrical/laser_ct_pcb/LEDs.sch (KiCad schematic (older format))
At the start: 8 parts

Commit message: End of episode 11.
Parts:
- added H1, H2: MountingHole_Pad, MountingHole:MountingHole_3.5mm, symbol Mechanical:MountingHole_Pad
- D1, D2, D3, D4: footprint LED_THT:LED_D5.0mm -> laser_ct:LED_D5.0mm
Connections:
- net labels added: GND
- wire segments 16 -> 21
Changed lines of the file:
@@
 F 0 "D1" H 2643 1745 50  0000 C CNN
 F 1 "LED" H 2643 1836 50  0000 C CNN
-F 2 "LED_THT:LED_D5.0mm" H 2650 2000 50  0001 C CNN
+F 2 "laser_ct:LED_D5.0mm" H 2650 2000 50  0001 C CNN
 F 3 "~" H 2650 2000 50  0001 C CNN
 	1    2650 2000
@@
 F 0 "D2" H 2643 3245 50  0000 C CNN
 F 1 "LED" H 2643 3336 50  0000 C CNN
-F 2 "LED_THT:LED_D5.0mm" H 2650 3500 50  0001 C CNN
+F 2 "laser_ct:LED_D5.0mm" H 2650 3500 50  0001 C CNN
 F 3 "~" H 2650 3500 50  0001 C CNN
 	1    2650 3500
@@
 F 0 "D3" H 2643 4745 50  0000 C CNN
 F 1 "LED" H 2643 4836 50  0000 C CNN
-F 2 "LED_THT:LED_D5.0mm" H 2650 5000 50  0001 C CNN
+F 2 "laser_ct:LED_D5.0mm" H 2650 5000 50  0001 C CNN
 F 3 "~" H 2650 5000 50  0001 C CNN
 	1    2650 5000
@@
 F 0 "D4" H 2643 6245 50  0000 C CNN
 F 1 "LED" H 2643 6336 50  0000 C CNN
-F 2 "LED_THT:LED_D5.0mm" H 2650 6500 50  0001 C CNN
+F 2 "laser_ct:LED_D5.0mm" H 2650 6500 50  0001 C CNN
 F 3 "~" H 2650 6500 50  0001 C CNN
 	1    2650 6500
@@
 Text HLabel 3200 6500 2    50   Output ~ 0
 LED4
+$Comp
+L power:GND #PWR0168
+U 1 1 5D7D2B16
+P 5050 1750
+F 0 "#PWR0168" H 5050 1500 50  0001 C CNN
+F 1 "GND" H 5055 1577 50  0000 C CNN
+F 2 "" H 5050 1750 50  0001 C CNN
+F 3 "" H 5050 1750 50  0001 C CNN
+	1    5050 1750
+	1    0    0    -1
+$EndComp
+$Comp
+L Mechanical:MountingHole_Pad H1
+U 1 1 5D7D3748
+P 4550 1350
+F 0 "H1" H 4650 1399 50  0000 L CNN
+F 1 "MountingHole_Pad" H 4650 1308 50  0000 L CNN
+F 2 "MountingHole:MountingHole_3.5mm" H 4550 1350 50  0001 C CNN
+F 3 "~" H 4550 1350 50  0001 C CNN
+	1    4550 1350
+	1    0    0    -1
+$EndComp
+$Comp
+L Mechanical:MountingHole_Pad H2
+U 1 1 5D7D552C
+P 5550 1350
+F 0 "H2" H 5650 1399 50  0000 L CNN
+F 1 "MountingHole_Pad" H 5650 1308 50  0000 L CNN
+F 2 "MountingHole:MountingHole_3.5mm" H 5550 1350 50  0001 C CNN
+F 3 "~" H 5550 1350 50  0001 C CNN
+	1    5550 1350
+	1    0    0    -1
+$EndComp
+Wire Wire Line
+	4550 1450 4550 1650
+Wire Wire Line
+	4550 1650 5050 1650
+Connection ~ 5050 1650
+Wire Wire Line
+	5050 1650 5550 1650
+Wire Wire Line
+	5550 1450 5550 1650
+Wire Wire Line
+	5050 1750 5050 1650
 $EndSCHEMATC
