File: Electrical/laser_ct_pcb/laser_ct_pcb.kicad_pcb (KiCad board)
At the start: 2 copper layers, 250 x 125 mm, 51 parts, among them Q1 Q_Photo_NPN, Q10 Q_Photo_NPN, Q11 Q_Photo_NPN, Q12 Q_Photo_NPN, Q13 Q_Photo_NPN, Q14 Q_Photo_NPN, Q15 Q_Photo_NPN, Q16 Q_Photo_NPN, Q17 Q_Photo_NPN, Q18 Q_Photo_NPN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

Commit message: End of episode 09.
Parts:
- added C1: 0.1uF, Capacitor_THT:CP_Radial_D5.0mm_P2.50mm, F.Cu at (92.5, 136.5)
- added C2: 10uF, Capacitor_THT:CP_Radial_D5.0mm_P2.50mm, F.Cu at (92.5, 130.0)
- added J1: Barrel_Jack_Switch, Connector_BarrelJack:BarrelJack_Horizontal, F.Cu at (81.0, 136.0)
- added U3: MIC29310-5.0WT, Package_TO_SOT_THT:TO-220-3_Horizontal_TabDown, F.Cu at (79.0, 130.0)
- moved Q23 263.8 mm to (210.5, 71.4), turned to 52.5 degrees
- moved R24 255.6 mm to (216.5, 80.5)
- moved R23 250.9 mm to (212.0, 85.5)
- moved Q24 244.6 mm to (214.3, 66.0), turned to 57.5 degrees
- moved R22 240.8 mm to (207.0, 91.0)
- moved R20 234.1 mm to (195.5, 100.5)
- moved Q22 233.4 mm to (206.2, 76.5), turned to 47.5 degrees
- moved R21 231.7 mm to (202.0, 96.5)
- moved R19 231.0 mm to (190.0, 103.5)
- moved Q21 224.4 mm to (201.5, 81.2), turned to 42.5 degrees
- moved Q19 222.3 mm to (191.0, 89.3), turned to 32.5 degrees
- moved Q18 215.8 mm to (185.2, 92.6), turned to 27.5 degrees
- moved Q15 213.5 mm to (166.5, 99.4), turned to 12.5 degrees
- moved Q20 212.9 mm to (196.4, 85.5), turned to 37.5 degrees
- moved R17 210.6 mm to (178.0, 109.5)
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Connections:
- A1 pad 19: Net-(A1-Pad19) -> /Phototransistors/PT24
- A1 pad 20: Net-(A1-Pad20) -> /Phototransistors/PT23
- A1 pad 21: Net-(A1-Pad21) -> /Phototransistors/PT22
- A1 pad 22: Net-(A1-Pad22) -> /Phototransistors/PT21
- A1 pad 23: Net-(A1-Pad23) -> /Phototransistors/PT20
- A1 pad 24: Net-(A1-Pad24) -> /Phototransistors/PT19
- A1 pad 25: Net-(A1-Pad25) -> /Phototransistors/PT18
- A1 pad 26: Net-(A1-Pad26) -> /Phototransistors/PT17
- Q10 pad 1: /Phototransistors/PT4 -> /PT10
- Q11 pad 1: /Phototransistors/PT14 -> /PT11
- Q12 pad 1: /Phototransistors/PT24 -> /PT12
- Q13 pad 1: /Phototransistors/PT5 -> /PT13
- Q14 pad 1: /Phototransistors/PT15 -> /PT14
- Q15 pad 1: /Phototransistors/PT6 -> /PT15
- Q16 pad 1: /Phototransistors/PT16 -> /PT16
- Q17 pad 1: /Phototransistors/PT7 -> /Phototransistors/PT17
- Q18 pad 1: /Phototransistors/PT17 -> /Phototransistors/PT18
- Q19 pad 1: /Phototransistors/PT8 -> /Phototransistors/PT19
- Q2 pad 1: /Phototransistors/PT11 -> /PT2
- Q20 pad 1: /Phototransistors/PT18 -> /Phototransistors/PT20
- Q21 pad 1: /Phototransistors/PT9 -> /Phototransistors/PT21
- Q22 pad 1: /Phototransistors/PT19 -> /Phototransistors/PT22
- Q23 pad 1: /Phototransistors/PT10 -> /Phototransistors/PT23
- Q24 pad 1: /Phototransistors/PT20 -> /Phototransistors/PT24
- Q3 pad 1: /Phototransistors/PT21 -> /PT3
- Q4 pad 1: /Phototransistors/PT2 -> /PT4
- Q5 pad 1: /Phototransistors/PT12 -> /PT5
- Q6 pad 1: /Phototransistors/PT22 -> /PT6
- Q7 pad 1: /Phototransistors/PT3 -> /PT7
- Q8 pad 1: /Phototransistors/PT13 -> /PT8
- Q9 pad 1: /Phototransistors/PT23 -> /Phototransistors/PT9
- R10 pad 2: /Phototransistors/PT4 -> /PT10
- R11 pad 2: /Phototransistors/PT14 -> /PT11
- R12 pad 2: /Phototransistors/PT24 -> /PT12
- R13 pad 2: /Phototransistors/PT5 -> /PT13
- R14 pad 2: /Phototransistors/PT15 -> /PT14
- R15 pad 2: /Phototransistors/PT6 -> /PT15
- R16 pad 2: /Phototransistors/PT16 -> /PT16
- R17 pad 2: /Phototransistors/PT7 -> /Phototransistors/PT17
- R18 pad 2: /Phototransistors/PT17 -> /Phototransistors/PT18
- R19 pad 2: /Phototransistors/PT8 -> /Phototransistors/PT19
- R2 pad 2: /Phototransistors/PT11 -> /PT2
- R20 pad 2: /Phototransistors/PT18 -> /Phototransistors/PT20
- R21 pad 2: /Phototransistors/PT9 -> /Phototransistors/PT21
- R22 pad 2: /Phototransistors/PT19 -> /Phototransistors/PT22
- R23 pad 2: /Phototransistors/PT10 -> /Phototransistors/PT23
- R24 pad 2: /Phototransistors/PT20 -> /Phototransistors/PT24
- R3 pad 2: /Phototransistors/PT21 -> /PT3
- R4 pad 2: /Phototransistors/PT2 -> /PT4
- R5 pad 2: /Phototransistors/PT12 -> /PT5
- R6 pad 2: /Phototransistors/PT22 -> /PT6
- R7 pad 2: /Phototransistors/PT3 -> /PT7
- R8 pad 2: /Phototransistors/PT13 -> /PT8
- R9 pad 2: /Phototransistors/PT23 -> /Phototransistors/PT9
- U1 pad 1: Net-(U1-Pad1) -> /PT8
- U1 pad 2: Net-(U1-Pad2) -> /PT7
- U1 pad 3: Net-(U1-Pad3) -> /PT6
- U1 pad 4: Net-(U1-Pad4) -> /PT5
- U1 pad 5: Net-(U1-Pad5) -> /PT4
- U1 pad 6: Net-(U1-Pad6) -> /PT3
- U1 pad 7: Net-(U1-Pad7) -> /PT2
- U1 pad 8: Net-(U1-Pad8) -> /Phototransistors/PT1
- U2 pad 1: Net-(U2-Pad1) -> /PT16
- U2 pad 2: Net-(U2-Pad2) -> /PT15
- U2 pad 3: Net-(U2-Pad3) -> /PT14
- U2 pad 4: Net-(U2-Pad4) -> /PT13
- U2 pad 5: Net-(U2-Pad5) -> /PT12
- U2 pad 6: Net-(U2-Pad6) -> /PT11
- U2 pad 7: Net-(U2-Pad7) -> /PT10
- U2 pad 8: Net-(U2-Pad8) -> /Phototransistors/PT9
Routing:
- net Net-(A1-Pad16): track 0.00 -> 127.4 mm, vias 0 -> 2
- net Net-(A1-Pad15): track 0.00 -> 109.0 mm, vias 0 -> 2
- net Net-(A1-Pad14): track 0.00 -> 106.1 mm
- net Net-(A1-Pad13): track 0.00 -> 94.3 mm, vias 0 -> 2
- net /Phototransistors/PT24: track 0.00 -> 76.6 mm
- net /Phototransistors/PT1: track 0.00 -> 69.9 mm
- net /Phototransistors/PT23: track 0.00 -> 68.7 mm
- net /PT2: track 0.00 -> 62.8 mm
- net /Phototransistors/PT22: track 0.00 -> 62.5 mm
- net /Phototransistors/PT17: track 0.00 -> 57.1 mm
- net /Phototransistors/PT21: track 0.00 -> 57.0 mm
- net /PT3: track 0.00 -> 56.3 mm
- net /Phototransistors/PT18: track 0.00 -> 55.7 mm
- net /Phototransistors/PT19: track 0.00 -> 54.2 mm
- net /Phototransistors/PT20: track 0.00 -> 54.1 mm
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
Commit message: End of episode 10.
Parts:
- added M1: 28BYJ-48, Connector_JST:JST_XH_B5B-XH-AM_1x05_P2.50mm_Vertical, B.Cu at (116.0, 146.0)
- added U4: ULN2003A, Package_DIP:DIP-16_W7.62mm, F.Cu at (130.0, 146.0)
- moved U1 35.9 mm to (154.5, 121.0)
- moved U2 21.5 mm to (181.6, 121.0)
- moved C1 13.0 mm to (105.5, 136.5)
- moved C2 13.0 mm to (105.5, 130.0)
- moved J1 13.0 mm to (94.0, 136.0)
- moved U3 13.0 mm to (92.0, 130.0)
Connections:
- A1 pad 10: Net-(A1-Pad10) -> /M2
- A1 pad 11: Net-(A1-Pad11) -> /M1
- A1 pad 8: Net-(A1-Pad8) -> /M4
- A1 pad 9: Net-(A1-Pad9) -> /M3
Routing:
- net /M4: track 0.00 -> 72.2 mm
- net /M3: track 0.00 -> 69.9 mm
- net /M2: track 0.00 -> 68.2 mm
- net /M1: track 0.00 -> 66.5 mm
- net Net-(A1-Pad16): track 127.4 -> 75.9 mm
- net Net-(A1-Pad15): track 109.0 -> 58.0 mm, vias 2 -> 1
- net Net-(A1-Pad14): track 106.1 -> 60.9 mm, vias 0 -> 1
- net Net-(A1-Pad13): track 94.3 -> 64.8 mm, vias 2 -> 1
- net /PT5: track 44.9 -> 67.5 mm
- net /PT4: track 50.3 -> 71.3 mm
- net /PT7: track 35.2 -> 55.9 mm
- net /PT10: track 33.0 -> 52.6 mm
- net /PT3: track 56.3 -> 75.3 mm
- net /Phototransistors/PT9: track 38.0 -> 56.9 mm
- net /PT6: track 39.8 -> 58.5 mm
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
Commit message: Added LED indicators for motor coils.
Parts:
- added D1: LED, LED_THT:LED_D5.0mm, F.Cu at (137.0, 136.2)
- added D2: LED, LED_THT:LED_D5.0mm, F.Cu at (147.0, 136.2)
- added D3: LED, LED_THT:LED_D5.0mm, F.Cu at (157.0, 136.2)
- added D4: LED, LED_THT:LED_D5.0mm, F.Cu at (167.0, 136.2)
- added R25: R_US, Resistor_THT:R_Axial_DIN0204_L3.6mm_D1.6mm_P7.62mm_Horizontal, F.Cu at (143.0, 141.5)
- added R26: R_US, Resistor_THT:R_Axial_DIN0204_L3.6mm_D1.6mm_P7.62mm_Horizontal, F.Cu at (153.0, 141.5)
- added R27: R_US, Resistor_THT:R_Axial_DIN0204_L3.6mm_D1.6mm_P7.62mm_Horizontal, F.Cu at (163.0, 141.5)
- added R28: R_US, Resistor_THT:R_Axial_DIN0204_L3.6mm_D1.6mm_P7.62mm_Horizontal, F.Cu at (173.0, 141.5)
Connections:
- net Net-(M1-Pad1) renamed /A
- net Net-(M1-Pad2) renamed /B
- net Net-(M1-Pad3) renamed /C
- net Net-(M1-Pad4) renamed /D
Routing:
- net /D: track 17.0 -> 69.0 mm
- net /C: track 13.5 -> 54.5 mm
- net /B: track 9.93 -> 39.8 mm
- net /A: track 6.38 -> 26.0 mm
- net Net-(D4-Pad2): track 0.00 -> 4.44 mm
- net Net-(D3-Pad2): track 0.00 -> 4.44 mm
- net Net-(D2-Pad2): track 0.00 -> 4.44 mm
- net Net-(D1-Pad2): track 0.00 -> 4.44 mm
Other:
- board size 250 x 125 mm -> 140 x 88.6 mm

Commit message: End of episode 11.
Parts:
- added H1: MountingHole_Pad, MountingHole:MountingHole_3.5mm, F.Cu at (84.0, 146.0)
- added H2: MountingHole_Pad, MountingHole:MountingHole_3.5mm, F.Cu at (216.0, 146.0)
- A1: footprint Module:Arduino_Nano -> laser_ct:Arduino_Nano
- D1, D2, D3, D4: footprint LED_THT:LED_D5.0mm -> laser_ct:LED_D5.0mm
- J1: footprint Connector_BarrelJack:BarrelJack_Horizontal -> laser_ct:BarrelJack_Horizontal
- M1: footprint Connector_JST:JST_XH_B5B-XH-AM_1x05_P2.50mm_Vertical -> laser_ct:JST_XH_B5B-XH-AM_1x05_P2.50mm_Vertical
Connections:
- A1 pad 27: +5V -> Net-(A1-Pad27)
- A1 pad 30: Net-(A1-Pad30) -> +5V
- J1 pad 3: Net-(J1-Pad3) -> GND
Routing:
- net +5V: track 0.00 -> 532.0 mm, vias 0 -> 6
- net +VDC: track 0.00 -> 18.5 mm
- net /PT14: track 29.1 -> 34.3 mm
- net /PT11: track 41.8 -> 46.9 mm
- added copper zone on B.Cu, net GND
- added copper zone on F.Cu, net GND
